File: synth-bus/synth-bus.kicad_pcb (KiCad board)
At the start: 2 copper layers, 226.1 x 35.6 mm, 19 parts, among them J1 Screw_Terminal_01x06, J10 Conn_02x08_Row_Letter_Last, J11 Conn_02x08_Row_Letter_Last, J12 Conn_02x08_Row_Letter_Last, J13 Conn_02x08_Row_Letter_Last, J2 Conn_02x08_Row_Letter_Last, J3 Conn_02x08_Row_Letter_Last, J4 Conn_02x08_Row_Letter_Last, J5 Conn_02x08_Row_Letter_Last, J6 Conn_02x08_Row_Letter_Last, J7 Conn_02x08_Row_Letter_Last, J8 Conn_02x08_Row_Letter_Last, J9 Conn_02x08_Row_Letter_Last

Commit message: Bus layout
Parts:
- moved J11 158.8 mm to (358.1, 108.0)
- moved J9 148.6 mm to (332.7, 108.0)
- moved J6 138.4 mm to (307.3, 108.0)
- moved J3 128.3 mm to (281.9, 108.0)
- moved J8 34.3 mm to (180.3, 108.0)
- moved J10 24.3 mm to (203.2, 108.0)
- moved J7 16.5 mm to (154.9, 108.0)
- moved R3 15.3 mm to (66.0, 111.8), turned to 270 degrees
- moved J2 15.2 mm to (78.7, 108.0)
- moved R2 13.5 mm to (58.4, 111.8), turned to 270 degrees
- moved J12 10.9 mm to (231.1, 108.0)
- moved R1 7.31 mm to (62.2, 111.9), turned to 270 degrees
- moved J4 5.08 mm to (104.1, 108.0)
- moved J5 5.08 mm to (129.5, 108.0)
- moved J13 2.84 mm to (256.5, 108.0)
Other:
- board size 226.1 x 35.6 mm -> 325.1 x 33 mm

Commit message: Bus schema + layout (cont.)
Parts:
- J10, J11, J12, J13, J2, J3, J4, J5, J6, J7, J8, J9: footprint Connectors_Multicomp:Multicomp_MC9A12-1634_2x08x2.54mm_Straight -> Connector_Multicomp:Multicomp_MC9A12-1634_2x08_P2.54mm_Vertical
- moved R1 18.0 mm to (62.4, 94.0), turned to 0 degrees
- moved D1 13.7 mm to (55.9, 94.0), turned to 180 degrees
- moved R2 13.3 mm to (62.4, 99.1), turned to 0 degrees
- moved D3 9.11 mm to (55.9, 104.1), turned to 180 degrees
- moved R3 8.44 mm to (62.4, 104.1), turned to 0 degrees
- moved D2 5.20 mm to (56.4, 99.1)
- moved J10 2.54 mm to (205.7, 108.0)
Connections:
- J1 pad 1: GND -> -12V
- J1 pad 2: +5V -> GND
- J1 pad 4: -12V -> +5V
- J10 pad 1: (no net) -> -12V
- J10 pad 10: (no net) -> +12V
- J10 pad 11: (no net) -> +5V
- J10 pad 12: (no net) -> +5V
- J10 pad 13: (no net) -> CV
- J10 pad 14: (no net) -> CV
- J10 pad 15: (no net) -> GATE
- J10 pad 16: (no net) -> GATE
- J10 pad 2: (no net) -> -12V
- J10 pad 3: (no net) -> GND
- J10 pad 4: (no net) -> GND
- J10 pad 5: (no net) -> GND
- J10 pad 6: (no net) -> GND
- J10 pad 7: (no net) -> GND
- J10 pad 8: (no net) -> GND
- J10 pad 9: (no net) -> +12V
- J11 pad 1: (no net) -> -12V
- J11 pad 10: (no net) -> +12V
- J11 pad 11: (no net) -> +5V
- J11 pad 12: (no net) -> +5V
- J11 pad 13: (no net) -> CV
- J11 pad 14: (no net) -> CV
- J11 pad 15: (no net) -> GATE
- J11 pad 16: (no net) -> GATE
- J11 pad 2: (no net) -> -12V
- J11 pad 3: (no net) -> GND
- J11 pad 4: (no net) -> GND
- J11 pad 5: (no net) -> GND
- J11 pad 6: (no net) -> GND
- J11 pad 7: (no net) -> GND
- J11 pad 8: (no net) -> GND
- J11 pad 9: (no net) -> +12V
- J12 pad 1: (no net) -> -12V
- J12 pad 10: (no net) -> +12V
- J12 pad 11: (no net) -> +5V
- J12 pad 12: (no net) -> +5V
- J12 pad 13: (no net) -> CV
- J12 pad 14: (no net) -> CV
- J12 pad 15: (no net) -> GATE
- J12 pad 16: (no net) -> GATE
- J12 pad 2: (no net) -> -12V
- J12 pad 3: (no net) -> GND
- J12 pad 4: (no net) -> GND
- J12 pad 5: (no net) -> GND
- J12 pad 6: (no net) -> GND
- J12 pad 7: (no net) -> GND
- J12 pad 8: (no net) -> GND
- J12 pad 9: (no net) -> +12V
- J13 pad 1: (no net) -> -12V
- J13 pad 10: (no net) -> +12V
- J13 pad 11: (no net) -> +5V
- J13 pad 12: (no net) -> +5V
- J13 pad 13: (no net) -> CV
- J13 pad 14: (no net) -> CV
- J13 pad 15: (no net) -> GATE
- J13 pad 16: (no net) -> GATE
- J13 pad 2: (no net) -> -12V
- J13 pad 3: (no net) -> GND
- J13 pad 4: (no net) -> GND
- J13 pad 5: (no net) -> GND
- J13 pad 6: (no net) -> GND
- J13 pad 7: (no net) -> GND
- J13 pad 8: (no net) -> GND
- J13 pad 9: (no net) -> +12V
- J2 pad 1: (no net) -> -12V
- J2 pad 10: (no net) -> +12V
- J2 pad 11: (no net) -> +5V
- J2 pad 12: (no net) -> +5V
- J2 pad 13: (no net) -> CV
- J2 pad 14: (no net) -> CV
- J2 pad 15: (no net) -> GATE
- J2 pad 16: (no net) -> GATE
- J2 pad 2: (no net) -> -12V
- J2 pad 3: (no net) -> GND
- J2 pad 4: (no net) -> GND
- J2 pad 5: (no net) -> GND
- J2 pad 6: (no net) -> GND
- J2 pad 7: (no net) -> GND
- J2 pad 8: (no net) -> GND
- J2 pad 9: (no net) -> +12V
- J3 pad 1: (no net) -> -12V
- J3 pad 10: (no net) -> +12V
- J3 pad 11: (no net) -> +5V
- J3 pad 12: (no net) -> +5V
- J3 pad 13: (no net) -> CV
- J3 pad 14: (no net) -> CV
- J3 pad 15: (no net) -> GATE
- J3 pad 16: (no net) -> GATE
- J3 pad 2: (no net) -> -12V
- J3 pad 3: (no net) -> GND
- J3 pad 4: (no net) -> GND
- J3 pad 5: (no net) -> GND
- J3 pad 6: (no net) -> GND
- J3 pad 7: (no net) -> GND
- J3 pad 8: (no net) -> GND
- J3 pad 9: (no net) -> +12V
- J4 pad 1: (no net) -> -12V
- J4 pad 10: (no net) -> +12V
- J4 pad 11: (no net) -> +5V
- J4 pad 12: (no net) -> +5V
- J4 pad 13: (no net) -> CV
- J4 pad 14: (no net) -> CV
- J4 pad 15: (no net) -> GATE
- J4 pad 16: (no net) -> GATE
- J4 pad 2: (no net) -> -12V
- J4 pad 3: (no net) -> GND
- J4 pad 4: (no net) -> GND
- J4 pad 5: (no net) -> GND
- J4 pad 6: (no net) -> GND
- J4 pad 7: (no net) -> GND
- J4 pad 8: (no net) -> GND
- J4 pad 9: (no net) -> +12V
- J5 pad 1: (no net) -> -12V
- J5 pad 10: (no net) -> +12V
- J5 pad 11: (no net) -> +5V
- J5 pad 12: (no net) -> +5V
- J5 pad 13: (no net) -> CV
- J5 pad 14: (no net) -> CV
- J5 pad 15: (no net) -> GATE
- J5 pad 16: (no net) -> GATE
- J5 pad 2: (no net) -> -12V
- J5 pad 3: (no net) -> GND
- J5 pad 4: (no net) -> GND
- J5 pad 5: (no net) -> GND
- J5 pad 6: (no net) -> GND
- J5 pad 7: (no net) -> GND
- J5 pad 8: (no net) -> GND
- J5 pad 9: (no net) -> +12V
- J6 pad 1: (no net) -> -12V
- J6 pad 10: (no net) -> +12V
- J6 pad 11: (no net) -> +5V
- J6 pad 12: (no net) -> +5V
- J6 pad 13: (no net) -> CV
- J6 pad 14: (no net) -> CV
- J6 pad 15: (no net) -> GATE
- J6 pad 16: (no net) -> GATE
- J6 pad 2: (no net) -> -12V
- J6 pad 3: (no net) -> GND
- J6 pad 4: (no net) -> GND
- J6 pad 5: (no net) -> GND
- J6 pad 6: (no net) -> GND
- J6 pad 7: (no net) -> GND
- J6 pad 8: (no net) -> GND
- J6 pad 9: (no net) -> +12V
- J7 pad 1: (no net) -> -12V
- J7 pad 10: (no net) -> +12V
- J7 pad 11: (no net) -> +5V
- J7 pad 12: (no net) -> +5V
- J7 pad 13: (no net) -> CV
- J7 pad 14: (no net) -> CV
- J7 pad 15: (no net) -> GATE
- J7 pad 16: (no net) -> GATE
- J7 pad 2: (no net) -> -12V
- J7 pad 3: (no net) -> GND
- J7 pad 4: (no net) -> GND
- J7 pad 5: (no net) -> GND
- J7 pad 6: (no net) -> GND
- J7 pad 7: (no net) -> GND
- J7 pad 8: (no net) -> GND
- J7 pad 9: (no net) -> +12V
- J8 pad 1: (no net) -> -12V
- J8 pad 10: (no net) -> +12V
- J8 pad 11: (no net) -> +5V
- J8 pad 12: (no net) -> +5V
- J8 pad 13: (no net) -> CV
- J8 pad 14: (no net) -> CV
- J8 pad 15: (no net) -> GATE
- J8 pad 16: (no net) -> GATE
- J8 pad 2: (no net) -> -12V
- J8 pad 3: (no net) -> GND
- J8 pad 4: (no net) -> GND
- J8 pad 5: (no net) -> GND
- J8 pad 6: (no net) -> GND
- J8 pad 7: (no net) -> GND
- J8 pad 8: (no net) -> GND
- J8 pad 9: (no net) -> +12V
- J9 pad 1: (no net) -> -12V
- J9 pad 10: (no net) -> +12V
- J9 pad 11: (no net) -> +5V
- J9 pad 12: (no net) -> +5V
- J9 pad 13: (no net) -> CV
- J9 pad 14: (no net) -> CV
- J9 pad 15: (no net) -> GATE
- J9 pad 16: (no net) -> GATE
- J9 pad 2: (no net) -> -12V
- J9 pad 3: (no net) -> GND
- J9 pad 4: (no net) -> GND
- J9 pad 5: (no net) -> GND
- J9 pad 6: (no net) -> GND
- J9 pad 7: (no net) -> GND
- J9 pad 8: (no net) -> GND
- J9 pad 9: (no net) -> +12V
Routing:
- net -12V: track 0.00 -> 646.7 mm
- net GATE: track 0.00 -> 625.5 mm
- net +12V: track 0.00 -> 625.5 mm
- net CV: track 0.00 -> 623.4 mm
- net +5V: track 0.00 -> 623.4 mm
- added copper zone on F.Cu, net GND
Other:
- net class High Current added: clearance 0.2, trace_width 1.2, via_dia 0.8, via_drill 0.4

Commit message: Bus progress
Parts:
- D1, D2: footprint LEDs:LED_1206_HandSoldering -> LED_SMD:LED_0805_2012Metric_Pad1.15x1.40mm_HandSolder
- D3: footprint LEDs:LED_0805_HandSoldering -> LED_SMD:LED_0805_2012Metric_Pad1.15x1.40mm_HandSolder
- moved D3 11.7 mm to (64.8, 111.8)
- moved R3 10.7 mm to (69.8, 111.8)
- moved D1 9.25 mm to (64.8, 96.5), turned to 0 degrees
- moved D2 8.73 mm to (64.8, 101.6)
- moved R1 7.87 mm to (69.8, 96.5)
- moved R2 7.87 mm to (69.8, 101.6)
- moved J1 3.81 mm to (50.8, 111.8)
Routing:
- net -12V: track 646.7 -> 633.0 mm
- net +5V: track 623.4 -> 633.0 mm
- net +12V: track 625.5 -> 633.0 mm
- net CV: track 623.4 -> 628.4 mm
- net GATE: track 625.5 -> 630.5 mm
- net Net-(D3-Pad1): track 0.00 -> 2.95 mm
- net Net-(D2-Pad2): track 0.00 -> 2.95 mm
- net Net-(D1-Pad2): track 0.00 -> 2.95 mm
- net GND: track 0.00 -> 1.44 mm, vias 0 -> 1
- added copper zone on B.Cu, net GND
Other:
- board size 325.1 x 33 mm -> 335.3 x 33 mm
- board text added: "+12V"
- board text added: "+5V"
- board text added: "-12V"
- board text added: "0V"
- board text added: "CV"
- board text added: "Gate"

Commit message: Synth Bus Board finished
This version was just sent to JLCPCB as rev 0.
Parts:
- removed the J4 at (104.1, 108.0)
- removed the J9 at (332.7, 108.0)
- added J10: Conn_02x08_Row_Letter_Last, Connector_Multicomp:Multicomp_MC9A12-1634_2x08_P2.54mm_Vertical, F.Cu at (281.9, 108.0)
- added J13: Conn_02x08_Row_Letter_Last, Connector_Multicomp:Multicomp_MC9A12-1634_2x08_P2.54mm_Vertical, F.Cu at (358.1, 108.0)
- added Ref**: Val**, SynthBus:SynthBusArt, F.Cu at (200.7, 102.1)
- moved J3 177.8 mm to (104.1, 108.0)
- moved J6 127.0 mm to (180.3, 108.0)
- moved J12 101.6 mm to (332.7, 108.0)
- moved J11 50.8 mm to (307.3, 108.0)
- moved J8 50.8 mm to (231.1, 108.0)
- renumbered J5 to J4, J7 to J5, J10 to J7, J13 to J9
Other:
- board text added: "Bus Board Rev 0"
