File: synth-bus/synth-bus.sch (KiCad schematic (older format))
At the start: 19 parts, among them J1 Screw_Terminal_01x06, J10 Conn_02x08_Row_Letter_Last, J11 Conn_02x08_Row_Letter_Last, J12 Conn_02x08_Row_Letter_Last, J13 Conn_02x08_Row_Letter_Last, J2 Conn_02x08_Row_Letter_Last, J3 Conn_02x08_Row_Letter_Last, J4 Conn_02x08_Row_Letter_Last, J5 Conn_02x08_Row_Letter_Last, J6 Conn_02x08_Row_Letter_Last, J7 Conn_02x08_Row_Letter_Last, J8 Conn_02x08_Row_Letter_Last, J9 Conn_02x08_Row_Letter_Last

Commit message: Bus schema + layout (cont.)
Parts:
- J10, J11, J12, J13, J2, J3, J4, J5, J6, J7, J8, J9: footprint Connectors_Multicomp:Multicomp_MC9A12-1634_2x08x2.54mm_Straight -> Connector_Multicomp:Multicomp_MC9A12-1634_2x08_P2.54mm_Vertical; symbol Connector_Generic:Conn_02x08_Row_Letter_Last -> Connector_Generic:Conn_02x08_Odd_Even
Connections:
- net +12V: now also J10.10 (Pin_10), J10.9 (Pin_9), J11.10 (Pin_10), J11.9 (Pin_9), J12.10 (Pin_10), J12.9 (Pin_9), J13.10 (Pin_10), J13.9 (Pin_9), J2.10 (Pin_10), J2.9 (Pin_9), J3.10 (Pin_10), J3.9 (Pin_9), J4.10 (Pin_10), J4.9 (Pin_9), J5.10 (Pin_10), J5.9 (Pin_9), J6.10 (Pin_10), J6.9 (Pin_9), J7.10 (Pin_10), J7.9 (Pin_9), J8.10 (Pin_10), J8.9 (Pin_9), J9.10 (Pin_10), J9.9 (Pin_9); no longer J10.4a (Pin_4a), J10.4b (Pin_4b), J11.4a (Pin_4a), J11.4b (Pin_4b), J12.4a (Pin_4a), J12.4b (Pin_4b), J13.4a (Pin_4a), J13.4b (Pin_4b), J2.4a (Pin_4a), J2.4b (Pin_4b), J3.4a (Pin_4a), J3.4b (Pin_4b), J4.4a (Pin_4a), J4.4b (Pin_4b), J5.4a (Pin_4a), J5.4b (Pin_4b), J6.4a (Pin_4a), J6.4b (Pin_4b), J7.4a (Pin_4a), J7.4b (Pin_4b), J8.4a (Pin_4a), J8.4b (Pin_4b), J9.4a (Pin_4a), J9.4b (Pin_4b)
- net +5V: now also J1.4 (Pin_4), J10.11 (Pin_11), J10.12 (Pin_12), J11.11 (Pin_11), J11.12 (Pin_12), J12.11 (Pin_11), J12.12 (Pin_12), J13.11 (Pin_11), J13.12 (Pin_12), J2.11 (Pin_11), J2.12 (Pin_12), J3.11 (Pin_11), J3.12 (Pin_12), J4.11 (Pin_11), J4.12 (Pin_12), J5.11 (Pin_11), J5.12 (Pin_12), J6.11 (Pin_11), J6.12 (Pin_12), J7.11 (Pin_11), J7.12 (Pin_12), J8.11 (Pin_11), J8.12 (Pin_12), J9.11 (Pin_11), J9.12 (Pin_12); no longer J1.2 (Pin_2), J10.3a (Pin_3a), J10.3b (Pin_3b), J11.3a (Pin_3a), J11.3b (Pin_3b), J12.3a (Pin_3a), J12.3b (Pin_3b), J13.3a (Pin_3a), J13.3b (Pin_3b), J2.3a (Pin_3a), J2.3b (Pin_3b), J3.3a (Pin_3a), J3.3b (Pin_3b), J4.3a (Pin_3a), J4.3b (Pin_3b), J5.3a (Pin_3a), J5.3b (Pin_3b), J6.3a (Pin_3a), J6.3b (Pin_3b), J7.3a (Pin_3a), J7.3b (Pin_3b), J8.3a (Pin_3a), J8.3b (Pin_3b), J9.3a (Pin_3a), J9.3b (Pin_3b)
- net -12V: now also J1.1 (Pin_1), J10.1 (Pin_1), J10.2 (Pin_2), J11.1 (Pin_1), J11.2 (Pin_2), J12.1 (Pin_1), J12.2 (Pin_2), J13.1 (Pin_1), J13.2 (Pin_2), J2.1 (Pin_1), J2.2 (Pin_2), J3.1 (Pin_1), J3.2 (Pin_2), J4.1 (Pin_1), J4.2 (Pin_2), J5.1 (Pin_1), J5.2 (Pin_2), J6.1 (Pin_1), J6.2 (Pin_2), J7.1 (Pin_1), J7.2 (Pin_2), J8.1 (Pin_1), J8.2 (Pin_2), J9.1 (Pin_1), J9.2 (Pin_2); no longer J1.4 (Pin_4), J10.8a (Pin_8a), J10.8b (Pin_8b), J11.8a (Pin_8a), J11.8b (Pin_8b), J12.8a (Pin_8a), J12.8b (Pin_8b), J13.8a (Pin_8a), J13.8b (Pin_8b), J2.8a (Pin_8a), J2.8b (Pin_8b), J3.8a (Pin_8a), J3.8b (Pin_8b), J4.8a (Pin_8a), J4.8b (Pin_8b), J5.8a (Pin_8a), J5.8b (Pin_8b), J6.8a (Pin_8a), J6.8b (Pin_8b), J7.8a (Pin_8a), J7.8b (Pin_8b), J8.8a (Pin_8a), J8.8b (Pin_8b), J9.8a (Pin_8a), J9.8b (Pin_8b)
- net CV: now also J10.13 (Pin_13), J10.14 (Pin_14), J11.13 (Pin_13), J11.14 (Pin_14), J12.13 (Pin_13), J12.14 (Pin_14), J13.13 (Pin_13), J13.14 (Pin_14), J2.13 (Pin_13), J2.14 (Pin_14), J3.13 (Pin_13), J3.14 (Pin_14), J4.13 (Pin_13), J4.14 (Pin_14), J5.13 (Pin_13), J5.14 (Pin_14), J6.13 (Pin_13), J6.14 (Pin_14), J7.13 (Pin_13), J7.14 (Pin_14), J8.13 (Pin_13), J8.14 (Pin_14), J9.13 (Pin_13), J9.14 (Pin_14); no longer J10.2a (Pin_2a), J10.2b (Pin_2b), J11.2a (Pin_2a), J11.2b (Pin_2b), J12.2a (Pin_2a), J12.2b (Pin_2b), J13.2a (Pin_2a), J13.2b (Pin_2b), J2.2a (Pin_2a), J2.2b (Pin_2b), J3.2a (Pin_2a), J3.2b (Pin_2b), J4.2a (Pin_2a), J4.2b (Pin_2b), J5.2a (Pin_2a), J5.2b (Pin_2b), J6.2a (Pin_2a), J6.2b (Pin_2b), J7.2a (Pin_2a), J7.2b (Pin_2b), J8.2a (Pin_2a), J8.2b (Pin_2b), J9.2a (Pin_2a), J9.2b (Pin_2b)
- net GATE: now also J10.15 (Pin_15), J10.16 (Pin_16), J11.15 (Pin_15), J11.16 (Pin_16), J12.15 (Pin_15), J12.16 (Pin_16), J13.15 (Pin_15), J13.16 (Pin_16), J2.15 (Pin_15), J2.16 (Pin_16), J3.15 (Pin_15), J3.16 (Pin_16), J4.15 (Pin_15), J4.16 (Pin_16), J5.15 (Pin_15), J5.16 (Pin_16), J6.15 (Pin_15), J6.16 (Pin_16), J7.15 (Pin_15), J7.16 (Pin_16), J8.15 (Pin_15), J8.16 (Pin_16), J9.15 (Pin_15), J9.16 (Pin_16); no longer J10.1a (Pin_1a), J10.1b (Pin_1b), J11.1a (Pin_1a), J11.1b (Pin_1b), J12.1a (Pin_1a), J12.1b (Pin_1b), J13.1a (Pin_1a), J13.1b (Pin_1b), J2.1a (Pin_1a), J2.1b (Pin_1b), J3.1a (Pin_1a), J3.1b (Pin_1b), J4.1a (Pin_1a), J4.1b (Pin_1b), J5.1a (Pin_1a), J5.1b (Pin_1b), J6.1a (Pin_1a), J6.1b (Pin_1b), J7.1a (Pin_1a), J7.1b (Pin_1b), J8.1a (Pin_1a), J8.1b (Pin_1b), J9.1a (Pin_1a), J9.1b (Pin_1b)
- net GND: now also J1.2 (Pin_2), J10.3 (Pin_3), J10.4 (Pin_4), J10.5 (Pin_5), J10.6 (Pin_6), J10.7 (Pin_7), J10.8 (Pin_8), J11.3 (Pin_3), J11.4 (Pin_4), J11.5 (Pin_5), J11.6 (Pin_6), J11.7 (Pin_7), J11.8 (Pin_8), J12.3 (Pin_3), J12.4 (Pin_4), J12.5 (Pin_5), J12.6 (Pin_6), J12.7 (Pin_7), J12.8 (Pin_8), J13.3 (Pin_3), J13.4 (Pin_4), J13.5 (Pin_5), J13.6 (Pin_6), J13.7 (Pin_7), J13.8 (Pin_8), J2.3 (Pin_3), J2.4 (Pin_4), J2.5 (Pin_5), J2.6 (Pin_6), J2.7 (Pin_7), J2.8 (Pin_8), J3.3 (Pin_3), J3.4 (Pin_4), J3.5 (Pin_5), J3.6 (Pin_6), J3.7 (Pin_7), J3.8 (Pin_8), J4.3 (Pin_3), J4.4 (Pin_4), J4.5 (Pin_5), J4.6 (Pin_6), J4.7 (Pin_7), J4.8 (Pin_8), J5.3 (Pin_3), J5.4 (Pin_4), J5.5 (Pin_5), J5.6 (Pin_6), J5.7 (Pin_7), J5.8 (Pin_8), J6.3 (Pin_3), J6.4 (Pin_4), J6.5 (Pin_5), J6.6 (Pin_6), J6.7 (Pin_7), J6.8 (Pin_8), J7.3 (Pin_3), J7.4 (Pin_4), J7.5 (Pin_5), J7.6 (Pin_6), J7.7 (Pin_7), J7.8 (Pin_8), J8.3 (Pin_3), J8.4 (Pin_4), J8.5 (Pin_5), J8.6 (Pin_6), J8.7 (Pin_7), J8.8 (Pin_8), J9.3 (Pin_3), J9.4 (Pin_4), J9.5 (Pin_5), J9.6 (Pin_6), J9.7 (Pin_7), J9.8 (Pin_8); no longer J1.1 (Pin_1), J10.5a (Pin_5a), J10.5b (Pin_5b), J10.6a (Pin_6a), J10.6b (Pin_6b), J10.7a (Pin_7a), J10.7b (Pin_7b), J11.5a (Pin_5a), J11.5b (Pin_5b), J11.6a (Pin_6a), J11.6b (Pin_6b), J11.7a (Pin_7a), J11.7b (Pin_7b), J12.5a (Pin_5a), J12.5b (Pin_5b), J12.6a (Pin_6a), J12.6b (Pin_6b), J12.7a (Pin_7a), J12.7b (Pin_7b), J13.5a (Pin_5a), J13.5b (Pin_5b), J13.6a (Pin_6a), J13.6b (Pin_6b), J13.7a (Pin_7a), J13.7b (Pin_7b), J2.5a (Pin_5a), J2.5b (Pin_5b), J2.6a (Pin_6a), J2.6b (Pin_6b), J2.7a (Pin_7a), J2.7b (Pin_7b), J3.5a (Pin_5a), J3.5b (Pin_5b), J3.6a (Pin_6a), J3.6b (Pin_6b), J3.7a (Pin_7a), J3.7b (Pin_7b), J4.5a (Pin_5a), J4.5b (Pin_5b), J4.6a (Pin_6a), J4.6b (Pin_6b), J4.7a (Pin_7a), J4.7b (Pin_7b), J5.5a (Pin_5a), J5.5b (Pin_5b), J5.6a (Pin_6a), J5.6b (Pin_6b), J5.7a (Pin_7a), J5.7b (Pin_7b), J6.5a (Pin_5a), J6.5b (Pin_5b), J6.6a (Pin_6a), J6.6b (Pin_6b), J6.7a (Pin_7a), J6.7b (Pin_7b), J7.5a (Pin_5a), J7.5b (Pin_5b), J7.6a (Pin_6a), J7.6b (Pin_6b), J7.7a (Pin_7a), J7.7b (Pin_7b), J8.5a (Pin_5a), J8.5b (Pin_5b), J8.6a (Pin_6a), J8.6b (Pin_6b), J8.7a (Pin_7a), J8.7b (Pin_7b), J9.5a (Pin_5a), J9.5b (Pin_5b), J9.6a (Pin_6a), J9.6b (Pin_6b), J9.7a (Pin_7a), J9.7b (Pin_7b)

Commit message: Bus progress
Parts:
- D1, D2: footprint LEDs:LED_1206_HandSoldering -> LED_SMD:LED_0805_2012Metric_Pad1.15x1.40mm_HandSolder
- D3: footprint LEDs:LED_0805_HandSoldering -> LED_SMD:LED_0805_2012Metric_Pad1.15x1.40mm_HandSolder
- J1: footprint Connectors_Terminal_Blocks:TerminalBlock_bornier-6_P5.08mm -> TerminalBlock_Phoenix:TerminalBlock_Phoenix_MKDS-3-6-5.08_1x06_P5.08mm_Horizontal
- R1, R2, R3: footprint Resistors_SMD:R_0603_HandSoldering -> Resistor_SMD:R_0603_1608Metric_Pad1.05x0.95mm_HandSolder
Changed lines of the file:
@@
 F 0 "D1" V 1447 3778 50  0000 L CNN
 F 1 "LED" V 1538 3778 50  0000 L CNN
-F 2 "LEDs:LED_1206_HandSoldering" H 1500 3700 50  0001 C CNN
+F 2 "LED_SMD:LED_0805_2012Metric_Pad1.15x1.40mm_HandSolder" H 1500 3700 50  0001 C CNN
 F 3 "~" H 1500 3700 50  0001 C CNN
 	1    1500 3700
@@
 F 0 "D2" V 1747 3778 50  0000 L CNN
 F 1 "LED" V 1838 3778 50  0000 L CNN
-F 2 "LEDs:LED_1206_HandSoldering" H 1800 3700 50  0001 C CNN
+F 2 "LED_SMD:LED_0805_2012Metric_Pad1.15x1.40mm_HandSolder" H 1800 3700 50  0001 C CNN
 F 3 "~" H 1800 3700 50  0001 C CNN
 	1    1800 3700
@@
 F 0 "D3" V 2139 3583 50  0000 R CNN
 F 1 "LED" V 2048 3583 50  0000 R CNN
-F 2 "LEDs:LED_0805_HandSoldering" H 2100 3700 50  0001 C CNN
+F 2 "LED_SMD:LED_0805_2012Metric_Pad1.15x1.40mm_HandSolder" H 2100 3700 50  0001 C CNN
 F 3 "~" H 2100 3700 50  0001 C CNN
 	1    2100 3700
@@
 F 0 "R1" H 1570 4146 50  0000 L CNN
 F 1 "R" H 1570 4055 50  0000 L CNN
-F 2 "Resistors_SMD:R_0603_HandSoldering" V 1430 4100 50  0001 C CNN
+F 2 "Resistor_SMD:R_0603_1608Metric_Pad1.05x0.95mm_HandSolder" V 1430 4100 50  0001 C CNN
 F 3 "~" H 1500 4100 50  0001 C CNN
 	1    1500 4100
@@
 F 0 "R2" H 1870 4146 50  0000 L CNN
 F 1 "R" H 1870 4055 50  0000 L CNN
-F 2 "Resistors_SMD:R_0603_HandSoldering" V 1730 4100 50  0001 C CNN
+F 2 "Resistor_SMD:R_0603_1608Metric_Pad1.05x0.95mm_HandSolder" V 1730 4100 50  0001 C CNN
 F 3 "~" H 1800 4100 50  0001 C CNN
 	1    1800 4100
@@
 F 0 "R3" H 2170 4146 50  0000 L CNN
 F 1 "R" H 2170 4055 50  0000 L CNN
-F 2 "Resistors_SMD:R_0603_HandSoldering" V 2030 4100 50  0001 C CNN
+F 2 "Resistor_SMD:R_0603_1608Metric_Pad1.05x0.95mm_HandSolder" V 2030 4100 50  0001 C CNN
 F 3 "~" H 2100 4100 50  0001 C CNN
 	1    2100 4100
@@
 F 0 "J1" H 1118 2917 50  0000 C CNN
 F 1 "Screw_Terminal_01x06" H 1118 2826 50  0000 C CNN
-F 2 "Connectors_Terminal_Blocks:TerminalBlock_bornier-6_P5.08mm" H 1200 2500 50  0001 C CNN
+F 2 "TerminalBlock_Phoenix:TerminalBlock_Phoenix_MKDS-3-6-5.08_1x06_P5.08mm_Horizontal" H 1200 2500 50  0001 C CNN
 F 3 "~" H 1200 2500 50  0001 C CNN
 	1    1200 2500

Commit message: Synth Bus Board finished
This version was just sent to JLCPCB as rev 0.
Parts:
- renumbered J3 to J10, J6 to J11, J9 to J12, J11 to J13, J4 to J3, J5 to J4, J7 to J5, J8 to J6, J10 to J7, J12 to J8, J13 to J9
Changed lines of the file:
@@
 $EndComp
 $Comp
-L Connector_Generic:Conn_02x08_Odd_Even J3
+L Connector_Generic:Conn_02x08_Odd_Even J10
 U 1 1 5D5DB691
 P 4650 3800
-F 0 "J3" H 4700 4317 50  0000 C CNN
+F 0 "J10" H 4700 4317 50  0000 C CNN
 F 1 "Conn_02x08_Row_Letter_Last" H 4700 4226 50  0000 C CNN
 F 2 "Connector_Multicomp:Multicomp_MC9A12-1634_2x08_P2.54mm_Vertical" H 4650 3800 50  0001 C CNN
@@
 $EndComp
 $Comp
-L Connector_Generic:Conn_02x08_Odd_Even J6
+L Connector_Generic:Conn_02x08_Odd_Even J11
 U 1 1 5D5DB727
 P 6150 3800
-F 0 "J6" H 6200 4317 50  0000 C CNN
+F 0 "J11" H 6200 4317 50  0000 C CNN
 F 1 "Conn_02x08_Row_Letter_Last" H 6200 4226 50  0000 C CNN
 F 2 "Connector_Multicomp:Multicomp_MC9A12-1634_2x08_P2.54mm_Vertical" H 6150 3800 50  0001 C CNN
@@
 $EndComp
 $Comp
-L Connector_Generic:Conn_02x08_Odd_Even J9
+L Connector_Generic:Conn_02x08_Odd_Even J12
 U 1 1 5D5DB7BD
 P 7600 3800
-F 0 "J9" H 7650 4317 50  0000 C CNN
+F 0 "J12" H 7650 4317 50  0000 C CNN
 F 1 "Conn_02x08_Row_Letter_Last" H 7650 4226 50  0000 C CNN
 F 2 "Connector_Multicomp:Multicomp_MC9A12-1634_2x08_P2.54mm_Vertical" H 7600 3800 50  0001 C CNN
@@
 $EndComp
 $Comp
-L Connector_Generic:Conn_02x08_Odd_Even J4
+L Connector_Generic:Conn_02x08_Odd_Even J3
 U 1 1 5D612070
 P 4650 4900
-F 0 "J4" H 4700 5417 50  0000 C CNN
+F 0 "J3" H 4700 5417 50  0000 C CNN
 F 1 "Conn_02x08_Row_Letter_Last" H 4700 5326 50  0000 C CNN
 F 2 "Connector_Multicomp:Multicomp_MC9A12-1634_2x08_P2.54mm_Vertical" H 4650 4900 50  0001 C CNN
@@
 $EndComp
 $Comp
-L Connector_Generic:Conn_02x08_Odd_Even J7
+L Connector_Generic:Conn_02x08_Odd_Even J5
 U 1 1 5D612106
 P 6150 4900
-F 0 "J7" H 6200 5417 50  0000 C CNN
+F 0 "J5" H 6200 5417 50  0000 C CNN
 F 1 "Conn_02x08_Row_Letter_Last" H 6200 5326 50  0000 C CNN
 F 2 "Connector_Multicomp:Multicomp_MC9A12-1634_2x08_P2.54mm_Vertical" H 6150 4900 50  0001 C CNN
@@
 $EndComp
 $Comp
-L Connector_Generic:Conn_02x08_Odd_Even J10
+L Connector_Generic:Conn_02x08_Odd_Even J7
 U 1 1 5D61219C
 P 7600 4900
-F 0 "J10" H 7650 5417 50  0000 C CNN
+F 0 "J7" H 7650 5417 50  0000 C CNN
 F 1 "Conn_02x08_Row_Letter_Last" H 7650 5326 50  0000 C CNN
 F 2 "Connector_Multicomp:Multicomp_MC9A12-1634_2x08_P2.54mm_Vertical" H 7600 4900 50  0001 C CNN
@@
 $EndComp
 $Comp
-L Connector_Generic:Conn_02x08_Odd_Even J13
+L Connector_Generic:Conn_02x08_Odd_Even J9
 U 1 1 5D612232
 P 9050 4900
-F 0 "J13" H 9100 5417 50  0000 C CNN
+F 0 "J9" H 9100 5417 50  0000 C CNN
 F 1 "Conn_02x08_Row_Letter_Last" H 9100 5326 50  0000 C CNN
 F 2 "Connector_Multicomp:Multicomp_MC9A12-1634_2x08_P2.54mm_Vertical" H 9050 4900 50  0001 C CNN
@@
 	8750 3700 8650 3700
 $Comp
-L Connector_Generic:Conn_02x08_Odd_Even J12
+L Connector_Generic:Conn_02x08_Odd_Even J8
 U 1 1 5D5DB853
 P 9050 3800
-F 0 "J12" H 9100 4317 50  0000 C CNN
+F 0 "J8" H 9100 4317 50  0000 C CNN
 F 1 "Conn_02x08_Row_Letter_Last" H 9100 4226 50  0000 C CNN
 F 2 "Connector_Multicomp:Multicomp_MC9A12-1634_2x08_P2.54mm_Vertical" H 9050 3800 50  0001 C CNN
@@
 $EndComp
 $Comp
-L Connector_Generic:Conn_02x08_Odd_Even J11
+L Connector_Generic:Conn_02x08_Odd_Even J13
 U 1 1 5D5C9347
 P 9050 2700
-F 0 "J11" H 9100 3217 50  0000 C CNN
+F 0 "J13" H 9100 3217 50  0000 C CNN
 F 1 "Conn_02x08_Row_Letter_Last" H 9100 3126 50  0000 C CNN
 F 2 "Connector_Multicomp:Multicomp_MC9A12-1634_2x08_P2.54mm_Vertical" H 9050 2700 50  0001 C CNN
@@
 $EndComp
 $Comp
-L Connector_Generic:Conn_02x08_Odd_Even J8
+L Connector_Generic:Conn_02x08_Odd_Even J6
 U 1 1 5D5BE3EA
 P 7600 2700
-F 0 "J8" H 7650 3217 50  0000 C CNN
+F 0 "J6" H 7650 3217 50  0000 C CNN
 F 1 "Conn_02x08_Row_Letter_Last" H 7650 3126 50  0000 C CNN
 F 2 "Connector_Multicomp:Multicomp_MC9A12-1634_2x08_P2.54mm_Vertical" H 7600 2700 50  0001 C CNN
@@
 $EndComp
 $Comp
-L Connector_Generic:Conn_02x08_Odd_Even J5
+L Connector_Generic:Conn_02x08_Odd_Even J4
 U 1 1 5D5B741A
 P 6150 2700
-F 0 "J5" H 6200 3217 50  0000 C CNN
+F 0 "J4" H 6200 3217 50  0000 C CNN
 F 1 "Conn_02x08_Row_Letter_Last" H 6200 3126 50  0000 C CNN
 F 2 "Connector_Multicomp:Multicomp_MC9A12-1634_2x08_P2.54mm_Vertical" H 6150 2700 50  0001 C CNN

Commit message: Locked all pots and jacks
Parts:
- R1: value R -> 270
- R2, R3: value R -> 1k
Changed lines of the file:
@@
 EESchema Schematic File Version 4
-LIBS:synth-bus-cache
 EELAYER 30 0
 EELAYER END
@@
 P 1500 4100
 F 0 "R1" H 1570 4146 50  0000 L CNN
-F 1 "R" H 1570 4055 50  0000 L CNN
+F 1 "270" H 1570 4055 50  0000 L CNN
 F 2 "Resistor_SMD:R_0603_1608Metric_Pad1.05x0.95mm_HandSolder" V 1430 4100 50  0001 C CNN
 F 3 "~" H 1500 4100 50  0001 C CNN
@@
 P 1800 4100
 F 0 "R2" H 1870 4146 50  0000 L CNN
-F 1 "R" H 1870 4055 50  0000 L CNN
+F 1 "1k" H 1870 4055 50  0000 L CNN
 F 2 "Resistor_SMD:R_0603_1608Metric_Pad1.05x0.95mm_HandSolder" V 1730 4100 50  0001 C CNN
 F 3 "~" H 1800 4100 50  0001 C CNN
@@
 P 2100 4100
 F 0 "R3" H 2170 4146 50  0000 L CNN
-F 1 "R" H 2170 4055 50  0000 L CNN
+F 1 "1k" H 2170 4055 50  0000 L CNN
 F 2 "Resistor_SMD:R_0603_1608Metric_Pad1.05x0.95mm_HandSolder" V 2030 4100 50  0001 C CNN
 F 3 "~" H 2100 4100 50  0001 C CNN
